File: PCB/Flight controler.kicad_sch (KiCad schematic)
At the start: 46 parts, among them J1 USB_C_Receptacle_USB2.0_14P, J2 Conn_02x03_Odd_Even, J3 01x04 (expressLRS), J4 ESC connector, J5 Conn_01x02_Pin, Q1 MMBT2222A, SW1 SW_Push, U1 ICM-42688-P, U2 AP2112K-3.3, U3 MP2359DJ, U4 STM32F411CEUx, Y1 Crystal

Commit message: Finished the PCB tracing and arrangement
Parts:
- U3: footprint Package_TO_SOT_SMD:SOT-23 -> Package_TO_SOT_SMD:TSOT-23-6
- U4: footprint Package_QFP:LQFP-48_7x7mm_P0.5mm -> Package_DFN_QFN:QFN-48-1EP_7x7mm_P0.5mm_EP5.6x5.6mm
Connections:
- net bat+: now also F1.1, J5.1 (Pin_1)
Changed lines of the file:
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@@
 	(wire
 		(pts
+			(xy 40.64 138.43) (xy 39.37 138.43)
+		)
+		(stroke
+			(width 0)
+			(type default)
+		)
+	)
+	(wire
+		(pts
 			(xy 27.94 138.43) (xy 36.83 138.43)
 		)
@@
 	(wire
 		(pts
-			(xy 39.37 138.43) (xy 39.37 140.97)
+			(xy 40.64 138.43) (xy 40.64 140.97)
 		)
 		(stroke
@@
 	(wire
 		(pts
-			(xy 16.51 140.97) (xy 39.37 140.97)
+			(xy 16.51 140.97) (xy 40.64 140.97)
 		)
 		(stroke
@@
 		)
 	)
+	(label "bat+"
+		(at 40.64 138.43 0)
+		(effects
+			(font
+				(size 1.27 1.27)
+			)
+			(justify left bottom)
+		)
+	)
 	(label "R9"
 		(at 154.94 43.18 0)
@@
 			)
 		)
-		(property "Footprint" "Package_QFP:LQFP-48_7x7mm_P0.5mm"
+		(property "Footprint" "Package_DFN_QFN:QFN-48-1EP_7x7mm_P0.5mm_EP5.6x5.6mm"
 			(at 167.64 99.06 0)
 			(hide yes)
@@
 			)
 		)
-		(property "Footprint" "Package_TO_SOT_SMD:SOT-23"
+		(property "Footprint" "Package_TO_SOT_SMD:TSOT-23-6"
 			(at 35.56 157.48 0)
 			(hide yes)
